File: PCB Rev1/untitled.kicad_sch (KiCad schematic)
At the start: 5 parts, among them U3 AP22653QW6-7

Commit message: Added power filtering stage 1, DC->DC Buck
Parts:
- renumbered R1 to R5, R2 to R6
Changed lines of the file:
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@@
 (kicad_sch
-	(version 20231120)
+	(version 20250114)
 	(generator "eeschema")
-	(generator_version "8.0")
+	(generator_version "9.0")
 	(paper "A4")
 	(junction
@@
 		(on_board yes)
 		(dnp no)
-		(property "Reference" "#PWR03"
+		(property "Reference" "#PWR08"
 			(at 166.37 99.06 0)
 			(effects
@@
 			(project "Data Logger Rev1"
 				(path "/adf54578-0edd-4ea8-a516-35041fcd2885/1f4eef8a-98e8-4167-8e58-ac4ffd368a0f"
-					(reference "#PWR03")
+					(reference "#PWR08")
 					(unit 1)
 				)
@@
 		(dnp no)
 		(fields_autoplaced yes)
-		(property "Reference" "#PWR02"
+		(property "Reference" "#PWR07"
 			(at 176.53 96.52 0)
 			(effects
@@
 			(project "Data Logger Rev1"
 				(path "/adf54578-0edd-4ea8-a516-35041fcd2885/1f4eef8a-98e8-4167-8e58-ac4ffd368a0f"
-					(reference "#PWR02")
+					(reference "#PWR07")
 					(unit 1)
 				)
@@
 		(dnp no)
 		(fields_autoplaced yes)
-		(property "Reference" "#PWR01"
+		(property "Reference" "#PWR05"
 			(at 101.6 88.9 0)
 			(effects
@@
 			(project ""
 				(path "/adf54578-0edd-4ea8-a516-35041fcd2885/1f4eef8a-98e8-4167-8e58-ac4ffd368a0f"
-					(reference "#PWR01")
+					(reference "#PWR05")
 					(unit 1)
 				)
@@
 		(dnp no)
 		(fields_autoplaced yes)
-		(property "Reference" "#PWR07"
+		(property "Reference" "#PWR04"
 			(at 95.25 109.22 0)
 			(effects
@@
 			(project ""
 				(path "/adf54578-0edd-4ea8-a516-35041fcd2885/1f4eef8a-98e8-4167-8e58-ac4ffd368a0f"
-					(reference "#PWR07")
+					(reference "#PWR04")
 					(unit 1)
 				)
@@
 		(dnp no)
 		(fields_autoplaced yes)
-		(property "Reference" "R1"
+		(property "Reference" "R5"
 			(at 161.29 90.17 90)
 			(effects
@@
 			(project "Data Logger Rev1"
 				(path "/adf54578-0edd-4ea8-a516-35041fcd2885/1f4eef8a-98e8-4167-8e58-ac4ffd368a0f"
-					(reference "R1")
+					(reference "R5")
 					(unit 1)
 				)
@@
 		(dnp no)
 		(fields_autoplaced yes)
-		(property "Reference" "#PWR08"
+		(property "Reference" "#PWR06"
 			(at 107.95 109.22 0)
 			(effects
@@
 			(project "Data Logger Rev1"
 				(path "/adf54578-0edd-4ea8-a516-35041fcd2885/1f4eef8a-98e8-4167-8e58-ac4ffd368a0f"
-					(reference "#PWR08")
+					(reference "#PWR06")
 					(unit 1)
 				)
@@
 		(on_board yes)
 		(dnp no)
-		(property "Reference" "R2"
+		(property "Reference" "R6"
 			(at 161.29 101.6 90)
 			(effects
@@
 			(project "Data Logger Rev1"
 				(path "/adf54578-0edd-4ea8-a516-35041fcd2885/1f4eef8a-98e8-4167-8e58-ac4ffd368a0f"
-					(reference "R2")
+					(reference "R6")
 					(unit 1)
 				)
