File: PCB Rev1/GPS_Module.kicad_sch (KiCad schematic)
At the start: 6 parts, among them U7 LT3042EDD_PBF, U8 SAM-M10Q

Commit message: hey now, over under 5 more hours of work?
Parts:
- removed C11, C4: 4.7uF, symbol Device:C
- removed C3: 0.47uF, symbol Device:C
- removed R7: 33k, symbol Device:R_US
- removed U7: LT3042EDD_PBF, footprints:VREG_LT3042EDD_PBF, symbol LT3042EDD_PBF:LT3042EDD_PBF
Connections:
- net GND: no longer U8.1 (GND), U8.10 (GND), U8.11 (GND), U8.15 (GND), U8.16 (GND), U8.20 (GND), U8.4 (GND), U8.5 (GND), U8.6 (GND)
- new net: U8.1 (GND), U8.10 (GND), U8.11 (GND), U8.15 (GND), U8.16 (GND), U8.20 (GND), U8.4 (GND), U8.5 (GND), U8.6 (GND)
- no-connect marks 7 -> 6
