File: PCB Rev1/sd_card.kicad_sch (KiCad schematic)
At the start: 10 parts, among them J5 MICRO_SD, U6 AP22653QW6-7

Commit message: hey now, over under 5 more hours of work?
Parts:
- removed C13: 0.1uF, symbol Device:C
- removed C14: 10uF, symbol Device:C
- removed R13: 49.9k, symbol Device:R
- removed R14: 10k, symbol Device:R
- removed U6: AP22653QW6-7, footprints:SOT26-A1-AP22653Q_DIO, symbol voltage_switch:AP22653QW6-7
Connections:
- net +3.3V: now reaches J5.4 (VDD), R10.2, R11.1, R12.2, R9.2
Other:
- note removed: "what is going on here??"
- moved on the sheet: J5, R10, R11, R12, R9
