File: PCB Rev1/AP22653Q.kicad_sch (KiCad schematic)
At the start: 5 parts, among them J4 MICRO_SD

Commit message: added new files and switches, notes,tps
Parts:
- removed J4: MICRO_SD, footprints:104031-0811_MOL, symbol sd_card_holder:1040310811
- removed R10, R7, R8, R9: 10k, symbol Device:R
- added C14: 10uF, symbol Device:C
- added C15, C16: 0.1uF, symbol Device:C
- added R11: 10k, symbol Device:R_US
- added R12: 40k, symbol Device:R_US
- added U6: AP22653QW6-7, footprints:SOT26-A1-AP22653Q_DIO, symbol voltage_switch:AP22653QW6-7
Connections:
- net GND: now also C14.2, C15.2, C16.2, R12.2, U6.2 (gnd)
- new net: R12.1, U6.5 (ilim)
- new net: R11.2, U6.4 (*fault)
- new net EN: U6.3 (en)
- new net V_IN: C14.1, C15.1, R11.1, U6.1 (in)
- new net V_OUT: C16.1, U6.6 (out)
Other:
- title: Micro SD Card -> Enable Switch for GPS and SD Card

Commit message: rev 2 schematic with minor changes, final send out before layout
Parts:
- renumbered C14 to C17, C15 to C18, C16 to C19, U6 to U4
Changed lines of the file:
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@@
 		(dnp no)
 		(fields_autoplaced yes)
-		(property "Reference" "C15"
+		(property "Reference" "C18"
 			(at 114.3 104.1399 0)
 			(effects
@@
 			(project ""
 				(path "/adf54578-0edd-4ea8-a516-35041fcd2885/905a8709-dadb-438d-a64a-98151fb9a03c"
-					(reference "C15")
+					(reference "C18")
 					(unit 1)
 				)
@@
 		(dnp no)
 		(fields_autoplaced yes)
-		(property "Reference" "C14"
+		(property "Reference" "C17"
 			(at 101.6 104.1399 0)
 			(effects
@@
 			(project ""
 				(path "/adf54578-0edd-4ea8-a516-35041fcd2885/905a8709-dadb-438d-a64a-98151fb9a03c"
-					(reference "C14")
+					(reference "C17")
 					(unit 1)
 				)
@@
 		(dnp no)
 		(fields_autoplaced yes)
-		(property "Reference" "#PWR020"
+		(property "Reference" "#PWR017"
 			(at 146.05 124.46 0)
 			(effects
@@
 			(project ""
 				(path "/adf54578-0edd-4ea8-a516-35041fcd2885/905a8709-dadb-438d-a64a-98151fb9a03c"
-					(reference "#PWR020")
+					(reference "#PWR017")
 					(unit 1)
 				)
@@
 		(dnp no)
 		(fields_autoplaced yes)
-		(property "Reference" "C16"
+		(property "Reference" "C19"
 			(at 175.26 104.1399 0)
 			(effects
@@
 			(project ""
 				(path "/adf54578-0edd-4ea8-a516-35041fcd2885/905a8709-dadb-438d-a64a-98151fb9a03c"
-					(reference "C16")
+					(reference "C19")
 					(unit 1)
 				)
@@
 		(dnp no)
 		(fields_autoplaced yes)
-		(property "Reference" "U6"
+		(property "Reference" "U4"
 			(at 144.78 82.55 0)
 			(effects
@@
 			(project ""
 				(path "/adf54578-0edd-4ea8-a516-35041fcd2885/905a8709-dadb-438d-a64a-98151fb9a03c"
-					(reference "U6")
-					(unit 1)
-				)
+					(reference "U4")
+					(unit 1)
+				)

Commit message: added PCB rev2!
Parts:
- removed C17: 10uF, symbol Device:C
- removed C19: 0.1uF, symbol Device:C
- added C16: 10uF, Capacitor_SMD:C_0805_2012Metric, symbol Device:C
- added C18: 0.1uF, Capacitor_SMD:C_0603_1608Metric, symbol Device:C
- C17: renamed from C18; footprint (none) -> Capacitor_SMD:C_0603_1608Metric; Part # (none) -> C0603C104K8RACAUTO
- R11: footprint (none) -> Resistor_SMD:R_0603_1608Metric; Part # (none) -> RK73H1JTTD1002F
- R12: footprint (none) -> footprints:RESC1005X35N; Part # (none) -> RNCF0402BTE40K0
- U4: Part # (none) -> AP22653QW6-7
Connections:
- net GND: now also C16.2, C18.2
- net V_IN: now also C16.1
- net V_OUT: now also C18.1
