File: PCB Rev1/Data Logger Rev1.kicad_sch (KiCad schematic)
At the start: 20 parts, among them J1 Conn_01x02_Socket, J2 USB_B_Micro, J3 BATTERY_PLUG (JST CONNECTOR??)

Commit message: added PCB rev2!
Parts:
- removed D2: SP0503BAHTG, footprints:SOT143, symbol tvs:SP0503BAHTG
- removed TP1: D-, symbol Connector:TestPoint
- removed TP10: DAT3, symbol Connector:TestPoint
- removed TP11, TP14: TestPoint, symbol Connector:TestPoint
- removed TP2: DAT0, symbol Connector:TestPoint
- removed TP4: D+, symbol Connector:TestPoint
- removed TP5: DAT1, symbol Connector:TestPoint
- removed TP7: CLK, symbol Connector:TestPoint
- removed TP8: DAT2, symbol Connector:TestPoint
- removed TP9: CMD, symbol Connector:TestPoint
- added TP15: 3.3V, footprints:TP_245X165, symbol Connector:TestPoint
- D1: Part # (none) -> PTVS20VZ1USK
- J1: value Conn_01x02_Socket -> 12V_Tractor; footprint Connector_PinSocket_2.54mm:PinSocket_1x02_P2.54mm_Vertical -> footprints:PHOENIX_1725656; Part # (none) -> 1725656
- J2: Part # (none) -> 10118193-0001LF
- J3: value BATTERY_PLUG (JST CONNECTOR??) -> BATTERY_PLUG; footprint Connector_PinSocket_2.54mm:PinSocket_1x02_P2.54mm_Vertical -> footprints:PHOENIX_1725656; Part # (none) -> 1725656
- TP12: value TestPoint -> 5V; footprint (none) -> footprints:TP_245X165; Part # (none) -> rct-0c
- TP13: value TestPoint -> V_BAT; footprint (none) -> footprints:TP_245X165; Part # (none) -> rct-0c
- TP14: renamed from TP15; value V_OUT_BAT_IC -> V_BAT_IC; footprint (none) -> footprints:TP_245X165; Part # (none) -> rct-0c
- TP3, TP6: footprint (none) -> footprints:TP_245X165; Part # (none) -> rct-0c
Connections:
- net +5V: now also TP12.1; no longer TP13.1
- net LOAD_SHARING_&_BAT_CHRG/V_BAT renamed V_BAT
- net V_BAT: now also TP13.1; no longer TP12.1
- new net 5V_3.3V LDO/3.3V: TP15.1
Other:
- sheet 12V->5V BUCK renamed 12V_5V BUCK
- sheet 5V-3.7V -> 3.3V renamed 5V_3.3V LDO
- sheet ESP32-S3-MINI-1U ports: added 3.3V, IO19, IO20, IO3, IO34, IO35, IO36, IO37, IO38, IO39, IO40, IO41, IO42, IO45, IO46, IO5, IO6; removed 1SEC, CLK, CMD, D+, D-, DAT0, DAT1, DAT2, DAT3, EN, EXTINT, SW_DET
- moved on the sheet: J2, J3, TP14, TP3, TP6
