File: PCB Rev1/SAM-M10Q.kicad_sch (KiCad schematic)
At the start: 5 parts, among them U6 SAM-M10Q

Commit message: added PCB rev2!
Parts:
- removed C24: 1uF, symbol Device:C
- added C22: 10uF, Capacitor_SMD:C_0805_2012Metric, symbol Device:C
- C23: value 10uF -> 1uF; footprint (none) -> Capacitor_SMD:C_0603_1608Metric; Part # (none) -> LMK107BJ105KAHT
- FB1: footprint (none) -> Resistor_SMD:R_0603_1608Metric; Part # (none) -> MI0603L221R-10
- JP1: footprint Connector_PinHeader_2.54mm:PinHeader_1x02_P2.54mm_Vertical -> Jumper:SolderJumper-2_P1.3mm_Open_RoundedPad1.0x1.5mm
- U6: Part # (none) -> SAM-M10Q
Connections:
- net 3.3V: now also C22.1; no longer C23.1
- net GND: now also C22.2
- net at FB1.1, U6.17 (VCC), U6.2 (VCC_IO): now also C23.1
