File: PCB Rev1/battery_management.kicad_sch (KiCad schematic)
At the start: 12 parts, among them U4 MCP73871-2CCI_ML

Commit message: rev 2 schematic with minor changes, final send out before layout
Parts:
- added R3: 10k, symbol Device:R_US
- C9: renamed from C8; value 4.7uF -> 10uF
- renumbered C9 to C10, C10 to C11, D3 to D4, D4 to D5, D5 to D6, R3 to R2, U4 to U2
Connections:
- net GND: now also R3.2
- net at U2.12 (PROG3): now also R3.1
Other:
- note added: "derated caps > 10V"
- moved on the sheet: C9, R2

Commit message: added PCB rev2!
Parts:
- C10: renamed from C11; footprint (none) -> Capacitor_SMD:C_0603_1608Metric; Part # (none) -> LMK107BJ475KAHT
- C8: renamed from C9; footprint (none) -> Capacitor_SMD:C_0805_2012Metric; Part # (none) -> GCM21BR71A106KE22K
- C9: renamed from C10; footprint (none) -> Capacitor_SMD:C_0603_1608Metric; Part # (none) -> LMK107BJ475KAHT
- D4: footprint (none) -> LED_SMD:LED_0603_1608Metric; Color (none) -> AMBER; Part # (none) -> 150060AS75000; Sim pins (none) -> 1=K 2=A
- D5: footprint (none) -> LED_SMD:LED_0603_1608Metric; Color (none) -> BLUE; Part # (none) -> 150080BS75000
- D6: footprint (none) -> LED_SMD:LED_0603_1608Metric; Color (none) -> GREEN; Part # (none) -> 150060GS75000
- R2: footprint (none) -> Resistor_SMD:R_0603_1608Metric; Part # (none) -> RK73H1JTTD1001F
- R3: footprint (none) -> Resistor_SMD:R_0603_1608Metric; Part # (none) -> RK73H1JTTD1002F
- R4, R5, R6: footprint (none) -> Resistor_SMD:R_0603_1608Metric; Part # (none) -> CRGCQ0603F470R
- TH1: footprint (none) -> Resistor_SMD:R_0402_1005Metric; Part # (none) -> NCU15XH103F6SRC
- U2: Part # (none) -> MCP73871-2CCI_ML
Other:
- note removed: "derated caps > 10V"
- note removed: "figure out colors"
- moved on the sheet: C8, C9, R2, R3
