File: PCB rev2/PCB Rev2.kicad_sch (KiCad schematic)
At the start: 11 parts, among them J1 12V_Tractor, J2 USB_B_Micro, J3 BATTERY_PLUG, U7 Value

Commit message: close to final, added PG pin
Parts:
- added J5: GPIO_BREAKOUT, footprints:PHOENIX_1725669, symbol Connector:Conn_01x03_Socket
- added LED1: XZCMECBDDGK53W, footprints:SON4_XZCME_SLD, symbol RGB_LED:XZCMECBDDGK53W
Connections:
- net GND: now also J5.1 (Pin_1)
- new net +3.3V: LED1.1
- new net ESP32-S3-MINI-1U/IO16: J5.2 (Pin_2)
- new net ESP32-S3-MINI-1U/IO17: J5.3 (Pin_3)
- new net ESP32-S3-MINI-1U/IO38: LED1.4
- new net ESP32-S3-MINI-1U/IO39: LED1.3
- new net ESP32-S3-MINI-1U/IO40: LED1.2
Other:
- sheet ESP32-S3-MINI-1U ports: added IO16, IO17, IO18; removed IO45, IO46
- sheet LOAD_SHARING_&_BAT_CHRG ports: added PG; removed none
