File: PCB rev2/PCB Rev2.kicad_sch (KiCad schematic)
At the start: 13 parts, among them J1 12V_Tractor, J2 USB_B_Micro, J3 BATTERY_PLUG, J5 GPIO_BREAKOUT, U7 Value

Commit message: Rev2 schematic/layout updates + Rev1 assets for full dev portability
Add custom KiCad symbol libs (Snapeda, TestPoint, greyscale_strawb),
footprints, DXF exports, Gerbers, schematic drawings, and Rev3 datasheet
draft. Update all Rev2 sub-schematics and PCB layout.

Co-Authored-By: Claude Sonnet 4.6 <noreply@anthropic.com>
Parts:
- J5: Part # (none) -> 1725669
- LED1: Part # (none) -> XZCMECBDDGK53W
- U7: value Value -> LORA; Part # (none) -> 114993390
