File: PCB rev2/mcu.kicad_sch (KiCad schematic)
At the start: 10 parts, among them U5 ESP32-S3-MINI-1U-N8

Commit message: Rev2 schematic/layout updates + Rev1 assets for full dev portability
Add custom KiCad symbol libs (Snapeda, TestPoint, greyscale_strawb),
footprints, DXF exports, Gerbers, schematic drawings, and Rev3 datasheet
draft. Update all Rev2 sub-schematics and PCB layout.

Co-Authored-By: Claude Sonnet 4.6 <noreply@anthropic.com>
Parts:
- BOOT1, RESET1: Part # (none) -> B3F-1000
