File: PCB rev2_revamped/battery_management.kicad_sch (KiCad schematic)
At the start: 8 parts, among them U2 MCP73871-2CCI_ML

Commit message: 0.8 edge clearance copper
Parts:
- TH1: LCSC (none) -> C333993
Changed lines of the file:
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@@
+			)
+		)
+		(property "LCSC" "C333993"
+			(at 95.25 116.84 90)
+			(effects
+				(font
+					(size 1.27 1.27)
+				)
+				(hide yes)
 			)
 		)
