File: PCB rev2_revamped/sd_card.kicad_sch (KiCad schematic)
At the start: 8 parts, among them J4 MICRO_SD

Commit message: final rev
Parts:
- removed J4: MICRO_SD, footprints:104031-0811_MOL, symbol sd_card_holder:1040310811
- added SIM1: C585350, EasyEDA_Lib:SIM-SMD_8P-1040310811, symbol EasyEDA_Lib:1040310811
Connections:
- net 3.3V: now also SIM1.4 (VDD)
- net CLK: now also SIM1.5 (CLK)
- net CMD: now also SIM1.3 (CMD)
- net DAT0: now also SIM1.7 (DAT0)
- net DAT1: now also SIM1.8 (DAT1)
- net DAT2: now also SIM1.1 (DAT2)
- net DAT3: now also SIM1.2 (CD/DAT3)
- net GND: now also SIM1.10, SIM1.11, SIM1.12, SIM1.13, SIM1.14, SIM1.6 (VSS), SIM1.9
- no-connect marks 0 -> 1
